File: DemoBoard/DemoBoard.kicad_sch (KiCad schematic)
At the start: 22 parts, among them J1 Conn_Coaxial, J2 Conn_01x02, J3 Conn_Coaxial, J4 Conn_Coaxial, J5 Conn_Coaxial, Q1 2N3904, U1 ICM7555xP, U101 ICM7555xP

Commit message: Sectioned Everything on PCB
Drew Traces and such
Parts:
- C1, C2, C3, C4: footprint (none) -> Capacitor_SMD:C_0805_2012Metric; LCSC# (none) -> C28323
- C5: footprint (none) -> Capacitor_SMD:C_0805_2012Metric; LCSC# (none) -> C49678
- D1(5.1V)1: LCSC# (none) -> C7441074
- D1(5.1V)2: renamed from D1(5.1V); LCSC# (none) -> C7441074
- Q1: LCSC# (none) -> C50176433
- R1, R3: footprint (none) -> Resistor_SMD:R_0805_2012Metric; LCSC# (none) -> C149504
- R2: footprint (none) -> Resistor_SMD:R_0805_2012Metric; LCSC# (none) -> C5555532
- R4: footprint (none) -> Resistor_SMD:R_0805_2012Metric; LCSC# (none) -> C17520
- R5: footprint (none) -> Capacitor_SMD:C_0805_2012Metric; LCSC# (none) -> C2933556
- TH1, TH2: footprint (none) -> Resistor_SMD:R_0805_2012Metric; LCSC# (none) -> C141588
Changed lines of the file:
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@@
 			)
 		)
-		(property "Footprint" ""
+		(property "Footprint" "Resistor_SMD:R_0805_2012Metric"
 			(at 41.402 92.71 90)
 			(effects
@@
 			)
 		)
+		(property "LCSC#" "C5555532"
+			(at 43.18 92.71 0)
+			(effects
+				(font
+					(size 1.27 1.27)
+				)
+				(hide yes)
+			)
+		)
 		(pin "2"
 		)
@@
 		(dnp no)
 		(fields_autoplaced yes)
-		(property "Reference" "D1(5.1V)"
+		(property "Reference" "D1(5.1V)2"
 			(at 45.72 102.8699 90)
 			(effects
@@
 			)
 		)
+		(property "LCSC#" "C7441074"
+			(at 43.18 104.14 90)
+			(effects
+				(font
+					(size 1.27 1.27)
+				)
+				(hide yes)
+			)
+		)
 		(pin "2"
 		)
@@
 			(project ""
 				(path "/894f620e-3404-4a40-a2a7-513bc1d5f99b"
-					(reference "D1(5.1V)")
+					(reference "D1(5.1V)2")
 					(unit 1)
 				)
@@
 			)
 		)
-		(property "Footprint" ""
+		(property "Footprint" "Capacitor_SMD:C_0805_2012Metric"
 			(at 31.4452 176.53 0)
 			(effects
@@
 			)
 		)
+		(property "LCSC#" "C28323"
+			(at 30.48 172.72 0)
+			(effects
+				(font
+					(size 1.27 1.27)
+				)
+				(hide yes)
+			)
+		)
 		(pin "2"
 		)
@@
 			)
 		)
-		(property "Footprint" ""
+		(property "Footprint" "Capacitor_SMD:C_0805_2012Metric"
 			(at 173.482 33.02 90)
 			(effects
@@
 			)
 		)
+		(property "LCSC#" "C2933556"
+			(at 175.26 33.02 0)
+			(effects
+				(font
+					(size 1.27 1.27)
+				)
+				(hide yes)
+			)
+		)
 		(pin "2"
 		)
@@
 			)
 		)
-		(property "Footprint" ""
+		(property "Footprint" "Resistor_SMD:R_0805_2012Metric"
 			(at 28.702 158.75 90)
 			(effects
@@
 			)
 		)
+		(property "LCSC#" "C149504"
+			(at 30.48 158.75 0)
+			(effects
+				(font
+					(size 1.27 1.27)
+				)
+				(hide yes)
+			)
+		)
 		(pin "2"
 		)
@@
 			)
 		)
-		(property "Footprint" ""
+		(property "Footprint" "Capacitor_SMD:C_0805_2012Metric"
 			(at 72.0852 182.88 0)
 			(effects
@@
 			)
 		)
+		(property "LCSC#" "C28323"
+			(at 71.12 179.07 0)
+			(effects
+				(font
+					(size 1.27 1.27)
+				)
+				(hide yes)
+			)
+		)
 		(pin "2"
 		)
@@
 			)
 		)
+		(property "LCSC#" "C7441074"
+			(at 81.28 179.07 90)
+			(effects
+				(font
+					(size 1.27 1.27)
+				)
+				(hide yes)
+			)
+		)
 		(pin "2"
 		)
@@
 			)
 		)
-		(property "Footprint" ""
+		(property "Footprint" "Capacitor_SMD:C_0805_2012Metric"
 			(at 176.2252 49.53 0)
 			(effects
@@
 			)
 		)
+		(property "LCSC#" "C49678"
+			(at 175.26 45.72 0)
+			(effects
+				(font
+					(size 1.27 1.27)
+				)
+				(hide yes)
+			)
+		)
 		(pin "2"
 		)
@@
 			)
 		)
+		(property "LCSC#" ""
+			(at 144.78 30.48 0)
+			(effects
+				(font
+					(size 1.27 1.27)
+				)
+				(hide yes)
+			)
+		)
 		(pin "1"
 		)
@@
 			)
 		)
-		(property "Footprint" ""
+		(property "Footprint" "Resistor_SMD:R_0805_2012Metric"
 			(at 30.48 146.05 0)
 			(effects
@@
 			)
 		)
+		(property "LCSC#" "C141588"
+			(at 30.48 146.05 0)
+			(effects
+				(font
+					(size 1.27 1.27)
+				)
+				(hide yes)
+			)
+		)
 		(pin "2"
 		)
@@
 			)
 		)
-		(property "Footprint" ""
+		(property "Footprint" "Resistor_SMD:R_0805_2012Metric"
 			(at 36.83 31.75 0)
 			(effects
@@
 			)
 		)
+		(property "LCSC#" "C141588"
+			(at 36.83 31.75 0)
+			(effects
+				(font
+					(size 1.27 1.27)
+				)
+				(hide yes)
+			)
+		)
 		(pin "2"
 		)
@@
 			)
 		)
-		(property "Footprint" ""
+		(property "Footprint" "Resistor_SMD:R_0805_2012Metric"
 			(at 35.052 41.91 90)
 			(effects
@@
 			)
 		)
+		(property "LCSC#" "C149504"
+			(at 36.83 41.91 0)
+			(effects
+				(font
+					(size 1.27 1.27)
+				)
+				(hide yes)
+			)
+		)
 		(pin "2"
 		)
@@
 			)
 		)
-		(property "Footprint" ""
+		(property "Footprint" "Capacitor_SMD:C_0805_2012Metric"
 			(at 33.9852 109.22 0)
 			(effects
@@
 			)
 		)
+		(property "LCSC#" "C28323"
+			(at 33.02 105.41 0)
+			(effects
+				(font
+					(size 1.27 1.27)
+				)
+				(hide yes)
+			)
+		)
 		(pin "2"
 		)
@@
 			)
 		)
-		(property "Footprint" ""
+		(property "Footprint" "Capacitor_SMD:C_0805_2012Metric"
 			(at 37.7952 59.69 0)
 			(effects
@@
 			)
 		)
+		(property "LCSC#" "C28323"
+			(at 36.83 55.88 0)
+			(effects
+				(font
+					(size 1.27 1.27)
+				)
+				(hide yes)
+			)
+		)
 		(pin "2"
 		)
@@
 			)
 		)
-		(property "Footprint" ""
+		(property "Footprint" "Resistor_SMD:R_0805_2012Metric"
 			(at 83.058 168.91 90)
 			(effects
@@
 			)
 		)
+		(property "LCSC#" "C17520"
+			(at 81.28 168.91 0)
+			(effects
+				(font
+					(size 1.27 1.27)
+				)
+				(hide yes)
+			)
+		)
 		(pin "2"
 		)
@@
 			(effects
 				(font
+					(size 1.27 1.27)
+				)
+				(hide yes)
+			)
+		)
+		(property "LCSC#" "C50176433"
+			(at 175.26 57.15 90)
+			(effects
+				(font
